Commit message: Add files via upload

File: description/robot.urdf.xacro (robot description, xacro)
@@ -1,7 +1,12 @@
 <?xml version="1.0"?>
 <robot xmlns:xacro="http://www.ros.org/wiki/xacro"  name="robot">
+    <xacro:arg name="use_ros2_control" default="true"/>
     <xacro:include filename="robot_core.xacro"/>
-    <!-- <xacro:include filename="gazebo_control.xacro"/> -->
-    <xacro:include filename="ros2_control.xacro"/>
+    <xacro:if value="$(arg use_ros2_control)">
+        <xacro:include filename="ros2_control.xacro"/>
+    </xacro:if>
+    <xacro:unless value="$(arg use_ros2_control)">
+        <xacro:include filename="gazebo_control.xacro"/>
+    </xacro:unless>
     <xacro:include filename="lidar.xacro"/>
     <xacro:include filename="camera.xacro"/>

File: description/robot_core.xacro (robot description, xacro)
@@ -3,8 +3,8 @@
     <link name="base_link"/>   <!--base_footprint -->
     <xacro:property name="base_constant" value="0.08333333333333333"/>
-    <xacro:property name="base_mass"     value="1.0"/>
-    <xacro:property name="base_width"    value="0.23"/>
+    <xacro:property name="base_mass"     value="4.0"/>
+    <xacro:property name="base_length"    value="0.23"/>
     <xacro:property name="base_height"   value="0.048"/>
-    <xacro:property name="base_depth"    value="0.16"/>
+    <xacro:property name="base_width"    value="0.16"/>
     <xacro:property name="wheel_constant"   value="0.08333333333333333"/>
     <xacro:property name="wheel_mass"       value="0.5"/>
@@ -16,12 +16,12 @@
             <mass value="5.0"/>
             <inertia
-                ixx="${base_constant * base_mass * (base_height*base_height + base_depth*base_depth)}" ixy="0.0" ixz="0.0"
-                iyy="${base_constant * base_mass * (base_width*base_width   + base_depth*base_depth)}" iyz="0.0"
-                izz="${base_constant * base_mass * (base_width*base_width   + base_height*base_height)}"/>
+                ixx="${base_constant * base_mass * (base_height*base_height + base_width*base_width)}" ixy="0.0" ixz="0.0"
+                iyy="${base_constant * base_mass * (base_length*base_length   + base_width*base_width)}" iyz="0.0"
+                izz="${base_constant * base_mass * (base_length*base_length   + base_height*base_height)}"/>
         </inertial>
         <visual name="">
             <origin xyz="0.0 0.0 0.0" rpy="0.0 0.0 0.0"/>
             <geometry>
-                <box size="0.23 0.16 0.048"/>
+                <box size="${base_length} ${base_width} ${base_height}"/> <!-- 0.23 0.16 0.048 -->
             </geometry>
             <material name="">
@@ -33,5 +33,5 @@
             <origin xyz="0.0 0.0 0.0" rpy="0.0 0.0 0.0"/>
             <geometry>
-                <box size="0.23 0.16 0.048"/>
+                <box size="${base_length} ${base_width} ${base_height}"/> <!-- 0.23 0.16 0.048 -->
             </geometry>
         </collision>
@@ -60,5 +60,5 @@
                 <origin xyz="0.0 0.0 0.0" rpy="0.0 0.0 0.0"/>
                 <geometry>
-                    <cylinder radius="0.0425" length="0.04"/>
+                    <cylinder radius="${wheel_radius}" length="0.04"/>
                 </geometry>
                 <material name="black">
@@ -69,5 +69,5 @@
                     <origin xyz="0.0 0.0 0.0" rpy="0.0 0.0 0.0"/>
                     <geometry>
-                        <cylinder radius="0.0425" length="0.04"/>
+                        <sphere radius="${wheel_radius}"/>
                     </geometry>
             </collision>

File: description/ros2_control.xacro (robot description, xacro)
@@ -5,41 +5,9 @@
             <plugin>gazebo_ros2_control/GazeboSystem</plugin>
         </hardware>
-        <!-- <joint name="wheel_front_left_joint">
-            <command_interface name="velocity">
-                <params name="min"> -10.0 </params>
-                <params name="max"> 10.0 </params>
-            </command_interface>
-            <state_interface name="velocity"/>
-            <state_interface name="position"/>
-        </joint>
-        <joint name="wheel_front_right_joint">
-            <command_interface name="velocity">
-                <params name="min"> -10.0 </params>
-                <params name="max"> 10.0 </params>
-            </command_interface>
-            <state_interface name="velocity"/>
-            <state_interface name="position"/>
-        </joint>
-        <joint name="wheel_rear_left_joint">
-            <command_interface name="velocity">
-                <params name="min"> -10.0 </params>
-                <params name="max"> 10.0 </params>
-            </command_interface>
-            <state_interface name="velocity"/>
-            <state_interface name="position"/>
-        </joint>
-        <joint name="wheel_rear_right_joint">
-            <command_interface name="velocity">
-                <params name="min"> -10.0 </params>
-                <params name="max"> 10.0 </params>
-            </command_interface>
-            <state_interface name="velocity"/>
-            <state_interface name="position"/>
-        </joint>  -->
         <xacro:macro name="define_wheel_joint" params="joint_name">
             <joint name="wheel_${joint_name}_joint">
                 <command_interface name="velocity">
-                    <params name="min">-10.0</params>
-                    <params name="max">10.0</params>
+                    <params name="min">-5.0</params>
+                    <params name="max">5.0</params>
                 </command_interface>
                 <state_interface name="velocity"/>
