Commit message: Add files via upload

File: description/lidar.xacro (robot description, xacro)
@@ -13,5 +13,5 @@
         <visual>
             <geometry>
-                <cylinder radius="0.05" length="0.04"/>
+                <cylinder radius="0.07" length="0.03"/>
             </geometry>
             <material name="">
@@ -22,15 +22,10 @@
         <collision>
             <geometry>
-                <cylinder radius="0.05" length="0.04"/>
+                <cylinder radius="0.07" length="0.03"/>
             </geometry>
         </collision>
-        <inertial>
-                <origin xyz="0.0 0.0 0.0" rpy="0.0 0.0 0.0"/>
-                <mass value="${wheel_mass}"/>
-                <inertia
-                    ixx="${wheel_constant * wheel_mass * (3 * wheel_radius * wheel_radius + wheel_height * wheel_height)}" ixy="0.0" ixz="0.0"
-                    iyy="${wheel_constant * wheel_mass * (3 * wheel_radius * wheel_radius + wheel_height * wheel_height)}" iyz="0.0"
-                    izz="${wheel_constant * wheel_mass * wheel_radius * wheel_radius}"/>
-        </inertial>
+        <xacro:inertial_cylinder mass="0.1" length="0.03" radius="0.07">
+            <origin xyz="0 0 0" rpy="0 0 0"/>
+        </xacro:inertial_cylinder>
     </link>
     <gazebo reference="laser_frame">

File: description/robot_core.xacro (robot description, xacro)
@@ -1,23 +1,22 @@
 <?xml version="1.0"?>
 <robot xmlns:xacro="http://www.ros.org/wiki/xacro">
+    <xacro:include filename="inertial_macros.xacro"/>
     <link name="base_link"/>   <!--base_footprint -->
-    <xacro:property name="base_constant" value="0.08333333333333333"/>
-    <xacro:property name="base_mass"     value="4.0"/>
-    <xacro:property name="base_length"    value="0.23"/>
-    <xacro:property name="base_height"   value="0.048"/>
-    <xacro:property name="base_width"    value="0.16"/>
-    <xacro:property name="wheel_constant"   value="0.08333333333333333"/>
-    <xacro:property name="wheel_mass"       value="0.5"/>
+    <!-- BASE_FOOTPRINT LINK -->
+    <joint name="base_footprint_joint" type="fixed">
+        <parent link="base_link"/>
+        <child link="base_footprint"/>
+        <origin xyz="0 0 0" rpy="0 0 0"/>
+    </joint>
+    <link name="base_footprint">
+    </link>
+    <xacro:property name="base_mass"        value="1.0"/>
+    <xacro:property name="base_length"      value="0.23"/>
+    <xacro:property name="base_height"      value="0.048"/>
+    <xacro:property name="base_width"       value="0.16"/>
+    <xacro:property name="wheel_mass"       value="0.06"/>
     <xacro:property name="wheel_radius"     value="0.0425"/>
-    <xacro:property name="wheel_height"     value="0.04"/>
+    <xacro:property name="wheel_thickness"  value="0.04"/>
     <link name="chassis">
-        <inertial>
-            <origin xyz="0.0 0.0 0.0" rpy="0.0 0.0 0.0"/>
-            <mass value="5.0"/>
-            <inertia
-                ixx="${base_constant * base_mass * (base_height*base_height + base_width*base_width)}" ixy="0.0" ixz="0.0"
-                iyy="${base_constant * base_mass * (base_length*base_length   + base_width*base_width)}" iyz="0.0"
-                izz="${base_constant * base_mass * (base_length*base_length   + base_height*base_height)}"/>
-        </inertial>
         <visual name="">
             <origin xyz="0.0 0.0 0.0" rpy="0.0 0.0 0.0"/>
@@ -36,4 +35,7 @@
             </geometry>
         </collision>
+        <xacro:inertial_box mass="0.5" x="${base_length}" y="${base_width}" z="${base_height}">
+            <origin xyz="${base_length/2} 0 ${base_height/2}" rpy="0 0 0"/>
+        </xacro:inertial_box>
     </link>
     <gazebo reference = "chassis">
@@ -49,12 +51,4 @@
     <xacro:macro name="wheel" params="name x y">
         <link name="wheel_${name}_link">
-            <inertial>
-                <origin xyz="0.0 0.0 0.0" rpy="0.0 0.0 0.0"/>
-                <mass value="${wheel_mass}"/>
-                <inertia
-                    ixx="${wheel_constant * wheel_mass * (3 * wheel_radius * wheel_radius + wheel_height * wheel_height)}" ixy="0.0" ixz="0.0"
-                    iyy="${wheel_constant * wheel_mass * (3 * wheel_radius * wheel_radius + wheel_height * wheel_height)}" iyz="0.0"
-                    izz="${wheel_constant * wheel_mass * wheel_radius * wheel_radius}"/>
-            </inertial>
             <visual name="">
                 <origin xyz="0.0 0.0 0.0" rpy="0.0 0.0 0.0"/>
@@ -72,4 +66,7 @@
                     </geometry>
             </collision>
+            <xacro:inertial_cylinder mass="${wheel_mass}" length="${wheel_thickness}" radius="${wheel_radius}">
+                <origin xyz="0 0 0" rpy="0 0 0"/>
+            </xacro:inertial_cylinder>
         </link>
         <gazebo reference = "wheel_${name}_link">
@@ -77,10 +74,10 @@
         </gazebo>
         <joint name="wheel_${name}_joint" type="continuous">
-            <origin xyz="${x} ${y} -0.007" rpy="1.57 0.0 0.0"/>
             <parent link="chassis"/>
             <child link="wheel_${name}_link"/>
+            <origin xyz="${x} ${y} -0.007" rpy="-1.57 0.0 0.0"/>
             <axis xyz=".0 .0 1.0"/>
-            <limit effort="10000" velocity="1000" />
-	        <dynamics damping="1.0" friction="1.0" />
+            <!-- <limit effort="10000" velocity="1000" /> -->
+	        <!-- <dynamics damping="1.0" friction="1.0" /> -->
         </joint>
     </xacro:macro>

File: description/ros2_control.xacro (robot description, xacro)
@@ -8,6 +8,6 @@
             <joint name="wheel_${joint_name}_joint">
                 <command_interface name="velocity">
-                    <params name="min">-5.0</params>
-                    <params name="max">5.0</params>
+                    <params name="min">-10.0</params>
+                    <params name="max">10.0</params>
                 </command_interface>
                 <state_interface name="velocity"/>
