Commit message: camera launch file

File: description/camera.xacro (robot description, xacro)
@@ -24,30 +24,25 @@
     <link name="camera_link_optical"> </link>
     <gazebo reference="camera_link">
-        <material>Gazebo/Red</material>
-        <!-- <sensor name="laser" type="ray">
+        <material>Gazebo/Black</material>
+        <sensor name="camera" type="camera">
             <pose> 0 0 0 0 0 0 </pose>
             <visualize>true</visualize>
             <update_rate>10</update_rate>
-            <ray>
-                <scan>
-                    <horizontal>
-                        <samples>360</samples>
-                        <min_angle>-3.14</min_angle>
-                        <max_angle>3.14</max_angle>
-                    </horizontal>
-                </scan>
-                <range>
-                    <min>0.3</min>
-                    <max>12</max>
-                </range>
-            </ray>
-            <plugin name="laser_controller" filename="libgazebo_ros_ray_sensor.so">
-                <ros>
-                    <argument>~/out:=scan</argument>
-                </ros>
-                <output_type>sensor_msgs/LaserScan</output_type>
-                <frame_name>laser_frame</frame_name>
+            <camera>
+                <horizontal_fov>1.089</horizontal_fov>
+                <image>
+                    <format>R8G8B8</format>
+                    <width>640</width>
+                    <height>480</height>
+                </image>
+                <clip>
+                    <near>0.05</near>
+                    <far>8.0</far>
+                </clip>
+            </camera>
+            <plugin name="camera_controller" filename="libgazebo_ros_camera.so">
+                <frame_name>camera_link_optical</frame_name>
             </plugin>
-            </sensor> -->
+        </sensor>
     </gazebo>
 </robot>

Commit message: Add files via upload

File: description/camera.xacro (robot description, xacro)
@@ -1,9 +1,4 @@
 <?xml version="1.0"?>
 <robot xmlns:xacro="http://www.ros.org/wiki/xacro">
-    <joint name="camera_joint" type="fixed">
-        <parent link="chassis"/>
-        <child link="camera_link"/>
-        <origin xyz="0.11 0 0.040" rpy="0 0 0"/>
-    </joint>
     <link name="camera_link">
         <visual>
@@ -17,4 +12,9 @@
         </visual>
     </link>
+    <joint name="camera_joint" type="fixed">
+        <parent link="chassis"/>
+        <child link="camera_link"/>
+        <origin xyz="${base_length/2} 0 ${base_height/2}" rpy="0 0 0"/>
+    </joint>
     <joint name="camera_optical_joint" type="fixed">
         <parent link="camera_link"/>

File: description/lidar.xacro (robot description, xacro)
@@ -1,17 +1,16 @@
 <?xml version="1.0"?>
 <robot xmlns:xacro="http://www.ros.org/wiki/xacro">
-    <xacro:property name="lidar_constant"   value="0.08333333333333333"/>
-    <xacro:property name="lidar_mass"       value="0.5"/>
+    <xacro:property name="lidar_mass"       value="0.010"/>
     <xacro:property name="lidar_radius"     value="0.0425"/>
-    <xacro:property name="lidar_height"     value="0.04"/>
+    <xacro:property name="lidar_height"     value="0.024"/>
     <joint name="laser_joint" type="fixed">
-        <parent link="chassis"/>
+        <parent link="lidar_base"/>
         <child link="laser_frame"/>
-        <origin xyz="-0.02 0.0 0.115" rpy="0.0 0.0 0.0"/>
+        <origin xyz="-0.00 0.0 0.035" rpy="0.0 0.0 0.0"/>
     </joint>
     <link name="laser_frame">
         <visual>
             <geometry>
-                <cylinder radius="0.07" length="0.03"/>
+                <cylinder radius="${lidar_radius}" length="${lidar_height}" />
             </geometry>
             <material name="">
@@ -22,8 +21,8 @@
         <collision>
             <geometry>
-                <cylinder radius="0.07" length="0.03"/>
+                <cylinder radius="${lidar_radius}" length="${lidar_height}" />
             </geometry>
         </collision>
-        <xacro:inertial_cylinder mass="0.1" length="0.03" radius="0.07">
+        <xacro:inertial_cylinder mass="${lidar_mass}" length="${lidar_height}" radius="${lidar_radius}">
             <origin xyz="0 0 0" rpy="0 0 0"/>
         </xacro:inertial_cylinder>

File: description/robot_core.xacro (robot description, xacro)
@@ -2,4 +2,7 @@
 <robot xmlns:xacro="http://www.ros.org/wiki/xacro">
     <xacro:include filename="inertial_macros.xacro"/>
+    <xacro:include filename="wheels.xacro"/>
+    <xacro:include filename="acrylic_base.xacro"/>
+    <xacro:include filename="stand_off.xacro"/>
     <link name="base_link"/>   <!--base_footprint -->
     <!-- BASE_FOOTPRINT LINK -->
@@ -18,9 +21,11 @@
     <xacro:property name="wheel_radius"     value="0.0425"/>
     <xacro:property name="wheel_thickness"  value="0.04"/>
+    <xacro:property name="acrylic_thickness"  value="0.003"/>
+    <xacro:property name="acrylic_width"  value="0.16"/>
     <link name="chassis">
         <visual name="">
-            <origin xyz="0.0 0.0 0.0" rpy="0.0 0.0 0.0"/>
+            <origin xyz="0 0 0"/>
             <geometry>
-                <box size="${base_length} ${base_width} ${base_height}"/> <!-- 0.23 0.16 0.048 -->
+                <box size="${base_length} ${base_width} ${base_height}"/> <!-- 0.23 0.16 0.048 ${base_height}-->
             </geometry>
             <material name="">
@@ -30,11 +35,11 @@
         </visual>
         <collision>
-            <origin xyz="0.0 0.0 0.0" rpy="0.0 0.0 0.0"/>
+            <origin xyz="0 0 0"/>
             <geometry>
                 <box size="${base_length} ${base_width} ${base_height}"/> <!-- 0.23 0.16 0.048 -->
             </geometry>
         </collision>
-        <xacro:inertial_box mass="0.5" x="${base_length}" y="${base_width}" z="${base_height}">
-            <origin xyz="${base_length/2} 0 ${base_height/2}" rpy="0 0 0"/>
+        <xacro:inertial_box mass="${base_mass}" x="${base_length}" y="${base_width}" z="${base_height}">  <!--mass="${base_mass}"-->
+            <origin xyz="0 0 0" rpy="0 0 0"/>
         </xacro:inertial_box>
     </link>
@@ -43,46 +48,21 @@
     </gazebo>
     <joint name="chassis_joint" type="fixed">
-        <origin xyz="0.0 0.0 0.0" rpy="0.0 0.0 0.0"/>
         <parent link="base_link"/>
         <child link="chassis"/>
-        <axis xyz="0.0 0.0 0.0"/>
+        <origin xyz="0.0 0.0 0.0425"/>
     </joint>
-    <!-- All Wheel links and joints -->
-    <xacro:macro name="wheel" params="name x y">
-        <link name="wheel_${name}_link">
-            <visual name="">
-                <origin xyz="0.0 0.0 0.0" rpy="0.0 0.0 0.0"/>
-                <geometry>
-                    <cylinder radius="${wheel_radius}" length="0.04"/>
-                </geometry>
-                <material name="black">
-                    <color rgba=".0 .0 0.0 1.0"/>
-                </material>
-            </visual>
-            <collision>
-                    <origin xyz="0.0 0.0 0.0" rpy="0.0 0.0 0.0"/>
-                    <geometry>
-                        <sphere radius="${wheel_radius}"/>
-                    </geometry>
-            </collision>
-            <xacro:inertial_cylinder mass="${wheel_mass}" length="${wheel_thickness}" radius="${wheel_radius}">
-                <origin xyz="0 0 0" rpy="0 0 0"/>
-            </xacro:inertial_cylinder>
-        </link>
-        <gazebo reference = "wheel_${name}_link">
-            <material>Gazebo/Black</material>
-        </gazebo>
-        <joint name="wheel_${name}_joint" type="continuous">
-            <parent link="chassis"/>
-            <child link="wheel_${name}_link"/>
-            <origin xyz="${x} ${y} -0.007" rpy="-1.57 0.0 0.0"/>
-            <axis xyz=".0 .0 1.0"/>
-            <!-- <limit effort="10000" velocity="1000" /> -->
-	        <!-- <dynamics damping="1.0" friction="1.0" /> -->
-        </joint>
-    </xacro:macro>
-    <xacro:wheel name="front_left"  x="0.085" y =" 0.105"/>
-    <xacro:wheel name="rear_left" x="-0.085" y =" 0.105"/>
-    <xacro:wheel name="rear_right"  x="-0.085" y =" -0.105"/>
-    <xacro:wheel name="front_right"   x="0.085" y =" -0.105"/>
+    <xacro:wheel name="front_left"  x="0.085" y =" 0.105" wheel_mass="${wheel_mass}" wheel_radius="${wheel_radius}" wheel_thickness="${wheel_thickness}"/>
+    <xacro:wheel name="rear_left" x="-0.085" y =" 0.105" wheel_mass="${wheel_mass}" wheel_radius="${wheel_radius}" wheel_thickness="${wheel_thickness}"/>
+    <xacro:wheel name="rear_right"  x="-0.085" y =" -0.105" wheel_mass="${wheel_mass}" wheel_radius="${wheel_radius}" wheel_thickness="${wheel_thickness}"/>
+    <xacro:wheel name="front_right"   x="0.085" y =" -0.105" wheel_mass="${wheel_mass}" wheel_radius="${wheel_radius}" wheel_thickness="${wheel_thickness}"/>
+    <xacro:acrylic_base parent="chassis" child="jetson_base" sheet_mass="0.02" sheet_length="0.190" sheet_width="${acrylic_width}" sheet_thickness="${acrylic_thickness}" xyz="-0.016 0 0.048"  />
+    <xacro:acrylic_base parent="chassis" child="lidar_base" sheet_mass="0.01" sheet_length="0.160" sheet_width="${acrylic_width}" sheet_thickness="${acrylic_thickness}" xyz="0 0 0.090" />
+    <xacro:robot_pillar parent="chassis" child="chassis_pillar1" standoff_mass="0.002" standoff_length="0.022" standoff_radius="0.003" xyz="0.06  0.07 0.036" />
+    <xacro:robot_pillar parent="chassis" child="chassis_pillar2" standoff_mass="0.002" standoff_length="0.022" standoff_radius="0.003" xyz="0.06  -0.07 0.036" />
+    <xacro:robot_pillar parent="chassis" child="chassis_pillar3" standoff_mass="0.002" standoff_length="0.022" standoff_radius="0.003" xyz="-0.06 0.07 0.036" />
+    <xacro:robot_pillar parent="chassis" child="chassis_pillar4" standoff_mass="0.002" standoff_length="0.022" standoff_radius="0.003" xyz="-0.06 -0.07 0.036" />
+    <xacro:robot_pillar parent="chassis" child="jetson_base_pillar1" standoff_mass="0.003" standoff_length="0.04" standoff_radius="0.003" xyz="0.06  0.07  0.07" />
+    <xacro:robot_pillar parent="chassis" child="jetson_base_pillar2" standoff_mass="0.003" standoff_length="0.04" standoff_radius="0.003" xyz="0.06  -0.07 0.07" />
+    <xacro:robot_pillar parent="chassis" child="jetson_base_pillar3" standoff_mass="0.003" standoff_length="0.04" standoff_radius="0.003" xyz="-0.06 0.07  0.07" />
+    <xacro:robot_pillar parent="chassis" child="jetson_base_pillar4" standoff_mass="0.003" standoff_length="0.04" standoff_radius="0.003" xyz="-0.06 -0.07 0.07" />
 </robot>
