Commit message: Add files via upload

File: description/acrylic_base.xacro (robot description, xacro)
@@ -8,6 +8,6 @@
                     <box size="${sheet_length} ${sheet_width} ${sheet_thickness}"/>
                 </geometry>
-                <material name="black">
-                    <color rgba="0.0 0.0 0.0 1.0"/>
+                <material name="darkgrey" >
+                    <color rgba="0.21176470588235294 0.21568627450980393 0.21568627450980393 1.0" />
                 </material>
             </visual>
@@ -27,5 +27,5 @@
         </joint>
         <gazebo reference = "${child}">
-            <material>Gazebo/Black</material>
+            <material>Gazebo/FlatBlack</material>
         </gazebo>
     </xacro:macro>

File: description/camera.xacro (robot description, xacro)
@@ -6,7 +6,6 @@
                 <box size="0.010 0.03 0.03"/>
             </geometry>
-            <material name="">
-                <color rgba="1.0 1.0 0.0 1.0"/>
-                <texture filename=""/>
+            <material name="darkgreyblue" >
+                <color rgba="0.1607843137254902 0.27450980392156865 0.3568627450980392 1.0" />
             </material>
         </visual>
@@ -15,5 +14,5 @@
         <parent link="chassis"/>
         <child link="camera_link"/>
-        <origin xyz="${base_length/2} 0 ${base_height/2}" rpy="0 0 0"/>
+        <origin xyz="${base_length/2} 0 ${(base_height/2) + 0.015}" rpy="0 0 0"/>
     </joint>
     <joint name="camera_optical_joint" type="fixed">
@@ -24,8 +23,8 @@
     <link name="camera_link_optical"> </link>
     <gazebo reference="camera_link">
-        <material>Gazebo/Black</material>
+        <material>Gazebo/DarkGrey</material>
         <sensor name="camera" type="camera">
             <pose> 0 0 0 0 0 0 </pose>
-            <visualize>true</visualize>
+            <visualize>false</visualize>
             <update_rate>10</update_rate>
             <camera>

File: description/lidar.xacro (robot description, xacro)
@@ -14,7 +14,6 @@
                 <cylinder radius="${lidar_radius}" length="${lidar_height}" />
             </geometry>
-            <material name="">
-                <color rgba="1.0 0.0 0.0 1.0"/>
-                <texture filename=""/>
+            <material name="darkgrey" >
+                <color rgba="0.21176470588235294 0.21568627450980393 0.21568627450980393 1.0" />
             </material>
         </visual>
@@ -29,8 +28,9 @@
     </link>
     <gazebo reference="laser_frame">
-        <material>Gazebo/Red</material>
+        <material>Gazebo/Grey</material>
         <sensor name="laser" type="ray">
             <pose> 0 0 0 0 0 0 </pose>
-            <visualize>true</visualize>
+            <visualize>false</visualize>
+            <!-- <visualize>true</visualize> -->
             <update_rate>10</update_rate>
             <ray>

File: description/robot.urdf.xacro (robot description, xacro)
@@ -2,4 +2,5 @@
 <robot xmlns:xacro="http://www.ros.org/wiki/xacro"  name="robot">
     <xacro:arg name="use_ros2_control" default="true"/>
+    <xacro:arg name="sim_mode" default="false"/>
     <xacro:include filename="robot_core.xacro"/>
     <xacro:if value="$(arg use_ros2_control)">

File: description/robot_core.xacro (robot description, xacro)
@@ -4,7 +4,7 @@
     <xacro:include filename="wheels.xacro"/>
     <xacro:include filename="acrylic_base.xacro"/>
-    <xacro:include filename="stand_off.xacro"/>
-    <link name="base_link"/>   <!--base_footprint -->
-    <!-- BASE_FOOTPRINT LINK -->
+    <xacro:include filename="standoff.xacro"/>
+    <link name="base_link"/>
+    <!--base_footprint -->
     <joint name="base_footprint_joint" type="fixed">
         <parent link="base_link"/>
@@ -23,13 +23,13 @@
     <xacro:property name="acrylic_thickness"  value="0.003"/>
     <xacro:property name="acrylic_width"  value="0.16"/>
+    <!--Main chassis -->
     <link name="chassis">
         <visual name="">
             <origin xyz="0 0 0"/>
             <geometry>
-                <box size="${base_length} ${base_width} ${base_height}"/> <!-- 0.23 0.16 0.048 ${base_height}-->
+                <box size="${base_length} ${base_width} ${base_height}"/>
             </geometry>
             <material name="">
                 <color rgba="1.0 1.0 0.0 1.0"/>
-                <texture filename=""/>
             </material>
         </visual>
@@ -37,8 +37,8 @@
             <origin xyz="0 0 0"/>
             <geometry>
-                <box size="${base_length} ${base_width} ${base_height}"/> <!-- 0.23 0.16 0.048 -->
+                <box size="${base_length} ${base_width} ${base_height}"/>
             </geometry>
         </collision>
-        <xacro:inertial_box mass="${base_mass}" x="${base_length}" y="${base_width}" z="${base_height}">  <!--mass="${base_mass}"-->
+        <xacro:inertial_box mass="${base_mass}" x="${base_length}" y="${base_width}" z="${base_height}">
             <origin xyz="0 0 0" rpy="0 0 0"/>
         </xacro:inertial_box>
@@ -52,10 +52,13 @@
         <origin xyz="0.0 0.0 0.0425"/>
     </joint>
+    <!-- Wheels -->
     <xacro:wheel name="front_left"  x="0.085" y =" 0.105" wheel_mass="${wheel_mass}" wheel_radius="${wheel_radius}" wheel_thickness="${wheel_thickness}"/>
     <xacro:wheel name="rear_left" x="-0.085" y =" 0.105" wheel_mass="${wheel_mass}" wheel_radius="${wheel_radius}" wheel_thickness="${wheel_thickness}"/>
     <xacro:wheel name="rear_right"  x="-0.085" y =" -0.105" wheel_mass="${wheel_mass}" wheel_radius="${wheel_radius}" wheel_thickness="${wheel_thickness}"/>
     <xacro:wheel name="front_right"   x="0.085" y =" -0.105" wheel_mass="${wheel_mass}" wheel_radius="${wheel_radius}" wheel_thickness="${wheel_thickness}"/>
+    <!-- Acrylic base -->
     <xacro:acrylic_base parent="chassis" child="jetson_base" sheet_mass="0.02" sheet_length="0.190" sheet_width="${acrylic_width}" sheet_thickness="${acrylic_thickness}" xyz="-0.016 0 0.048"  />
     <xacro:acrylic_base parent="chassis" child="lidar_base" sheet_mass="0.01" sheet_length="0.160" sheet_width="${acrylic_width}" sheet_thickness="${acrylic_thickness}" xyz="0 0 0.090" />
+    <!-- Standoffs -->
     <xacro:robot_pillar parent="chassis" child="chassis_pillar1" standoff_mass="0.002" standoff_length="0.022" standoff_radius="0.003" xyz="0.06  0.07 0.036" />
     <xacro:robot_pillar parent="chassis" child="chassis_pillar2" standoff_mass="0.002" standoff_length="0.022" standoff_radius="0.003" xyz="0.06  -0.07 0.036" />

File: description/ros2_control.xacro (robot description, xacro)
@@ -1,26 +1,49 @@
 <?xml version="1.0"?>
 <robot xmlns:xacro="http://www.ros.org/wiki/xacro">
-    <ros2_control name="GazeboSystem" type="system">
-        <hardware>
-            <plugin>gazebo_ros2_control/GazeboSystem</plugin>
-        </hardware>
-        <xacro:macro name="define_wheel_joint" params="joint_name">
-            <joint name="wheel_${joint_name}_joint">
-                <command_interface name="velocity">
-                    <params name="min">-10.0</params>
-                    <params name="max">10.0</params>
-                </command_interface>
-                <state_interface name="velocity"/>
-                <state_interface name="position"/>
-            </joint>
-        </xacro:macro>
-        <xacro:define_wheel_joint joint_name="front_left"/>
-        <xacro:define_wheel_joint joint_name="front_right"/>
-        <xacro:define_wheel_joint joint_name="rear_left"/>
-        <xacro:define_wheel_joint joint_name="rear_right"/>
-    </ros2_control>
+    <xacro:macro name="define_wheel_joint" params="joint_name">
+        <joint name="wheel_${joint_name}_joint">
+            <command_interface name="velocity">
+                <params name="min">-10.0</params>
+                <params name="max">10.0</params>
+            </command_interface>
+            <state_interface name="velocity"/>
+            <state_interface name="position"/>
+        </joint>
+    </xacro:macro>
+    <xacro:unless value="$(arg sim_mode)">
+        <ros2_control name="RealRobot" type="system">
+            <hardware>
+            <plugin>diffdrive_arduino/DiffDriveArduinoHardware</plugin>
+                <param name="wheel_front_left_joint">wheel_front_left_joint</param>
+                <param name="wheel_front_right_joint">wheel_front_right_joint</param>
+                <param name="wheel_rear_left_joint">wheel_rear_left_joint</param>
+                <param name="wheel_rear_right_joint">wheel_rear_right_joint</param>
+                <param name="loop_rate">30</param>
+                <param name="device">/dev/ttyUSB0</param>
+                <param name="baud_rate">57600</param>
+                <param name="timeout_ms">1000</param>
+                <param name="enc_counts_per_rev">19560</param>
+            </hardware>
+            <xacro:define_wheel_joint joint_name="front_left"/>
+            <xacro:define_wheel_joint joint_name="front_right"/>
+            <xacro:define_wheel_joint joint_name="rear_left"/>
+            <xacro:define_wheel_joint joint_name="rear_right"/>
+        </ros2_control>
+    </xacro:unless>
+    <xacro:if value="$(arg sim_mode)">
+        <ros2_control name="GazeboSystem" type="system">
+            <hardware>
+                <plugin>gazebo_ros2_control/GazeboSystem</plugin>
+            </hardware>
+            <xacro:define_wheel_joint joint_name="front_left"/>
+            <xacro:define_wheel_joint joint_name="front_right"/>
+            <xacro:define_wheel_joint joint_name="rear_left"/>
+            <xacro:define_wheel_joint joint_name="rear_right"/>
+        </ros2_control>
+    </xacro:if>
     <gazebo>
         <plugin name="gazebo_ros2_control" filename="libgazebo_ros2_control.so">
             <parameters>$(find rog_ros_bot)/config/my_controllers.yaml</parameters>
+            <parameters>$(find rog_ros_bot)/config/gaz_ros2_ctl_use_sim.yaml</parameters>
         </plugin>
     </gazebo>

File: description/wheels.xacro (robot description, xacro)
@@ -9,6 +9,6 @@
                     <cylinder radius="${wheel_radius}" length="${wheel_thickness}"/>
                 </geometry>
-                <material name="black">
-                    <color rgba="0.0 0.0 0.0 1.0"/>
+                <material name="almostblack" >
+                    <color rgba="0.027450980392156862 0.050980392156862744 0.050980392156862744 1.0" />
                 </material>
             </visual>
