Commit message: update

File: description/gazebo_control.xacro (robot description, xacro)
@@ -3,6 +3,29 @@
         <!--skid_steer_drive_controller-->
     <gazebo>
-        <plugin name="diff_drive" filename="libgazebo_ros_skid_steer_drive.so">
+        <plugin name="gazebo_ros_joint_state_publisher"
+            filename = "libgazebo_ros_joint_state_publisher.so">
+            <update_rate>20</update_rate>
+            <joint_name>wheel_front_left_joint</joint_name>
+            <joint_name>wheel_front_right_joint</joint_name>
+            <joint_name>wheel_rear_left_joint</joint_name>
+            <joint_name>wheel_rear_right_joint</joint_name>
+            <joint_name>wheel_rear_right_joint</joint_name>
+        </plugin>
+    </gazebo>
+    <gazebo>
+        <plugin name="gazebo_ros_joint_pose_trajectory"
+            filename = "libgazebo_ros_joint_pose_trajectory.so">
+            <update_rate>20</update_rate>
+            <joint_name>wheel_front_left_joint</joint_name>
+            <joint_name>wheel_front_right_joint</joint_name>
+            <joint_name>wheel_rear_left_joint</joint_name>
+            <joint_name>wheel_rear_right_joint</joint_name>
+            <joint_name>wheel_rear_right_joint</joint_name>
+        </plugin>
+    </gazebo>
+    <!-- <gazebo>
+        <plugin name="mobile_base_controller" filename="libgazebo_ros_skid_steer_drive.so">
             <updateRate>100.0</updateRate>
+            <robotNamespace>/armbot</robotNamespace>
             <leftFrontJoint>wheel_front_left_joint</leftFrontJoint>
             <rightFrontJoint>wheel_front_right_joint</rightFrontJoint>
@@ -11,12 +34,42 @@
             <wheelSeparation>0.16</wheelSeparation>
             <wheelDiameter>0.085</wheelDiameter>
-            <broadcastTF>true</broadcastTF>
-            <max_wheel_torque>200</max_wheel_torque>
-            <max_wheel_acceleration>10.0</max_wheel_acceleration>
-            <odometry_frame>odom</odometry_frame>
-            <robot_base_frame>chassis</robot_base_frame>
+            <robotBaseFrame>base_link</robotBaseFrame>
+            <torque>20</torque>
+            <commandTopic>mobile_base_controller/cmd_vel</commandTopic>
+            <odometryTopic>mobile_base_controller/odom</odometryTopic>
+            <odometryFrame>odom</odometryFrame>
             <publish_odom>true</publish_odom>
             <publish_odom_tf>true</publish_odom_tf>
             <publish_wheel_tf>true</publish_wheel_tf>
+            <covariance_x>100.0</covariance_x>
+            <covariance_y>100.0</covariance_y>
+            <covariance_yaw>100.0</covariance_yaw>
+            <odometryRate>20.0</odometryRate>
+            <broadcastTF>true</broadcastTF>
+        </plugin>
+    </gazebo> -->
+    <gazebo>
+        <plugin name="skid_steer_drive_controller" filename="libgazebo_ros_skid_steer_drive.so">
+            <updateRate>10.0</updateRate>
+            <robotNamespace>/</robotNamespace>
+            <leftFrontJoint>left_wheel_hinge_front</leftFrontJoint>
+            <rightFrontJoint>right_wheel_hinge_front</rightFrontJoint>
+            <leftRearJoint>left_wheel_hinge_back</leftRearJoint>
+            <rightRearJoint>right_wheel_hinge_back</rightRearJoint>
+            <wheelSeparation>0.4</wheelSeparation>
+            <wheelDiameter>0.2</wheelDiameter>
+            <robotBaseFrame>robot_footprint</robotBaseFrame>
+            <torque>10</torque>
+            <topicName>cmd_vel</topicName>
+            <odometryTopic>odom</odometryTopic>
+            <odometryFrame>odom</odometryFrame>
+            <commandTopic>cmd_vel</commandTopic>
+            <topic_name_twist>cmd_vel</topic_name_twist>
+            <topic_name_odometry>odom</topic_name_odometry>
+            <topic_name_joint>joint</topic_name_joint>
+            <broadcastTF>true</broadcastTF>
+            <covariance_x>0.0001</covariance_x>
+            <covariance_y>0.0001</covariance_y>
+            <covariance_yaw>0.01</covariance_yaw>
         </plugin>
     </gazebo>

File: description/robot.urdf.xacro (robot description, xacro)
@@ -2,5 +2,5 @@
 <robot xmlns:xacro="http://www.ros.org/wiki/xacro"  name="robot">
     <xacro:include filename="robot_core.xacro"/>
-    <!-- <xacro:include filename="gazebo_control.xacro"/> -->
+    <xacro:include filename="gazebo_control.xacro"/>
     <xacro:include filename="lidar.xacro"/>
     <xacro:include filename="camera.xacro"/>

File: description/robot_core.xacro (robot description, xacro)
@@ -77,4 +77,6 @@
             <child link="wheel_${name}_link"/>
             <axis xyz=".0 .0 1.0"/>
+            <limit effort="10000" velocity="1000" />
+	        <dynamics damping="1.0" friction="1.0" />
         </joint>
     </xacro:macro>
@@ -88,5 +90,5 @@
     <xacro:wheel name="front_left"  x="-0.085" y =" -0.105"/>
     <xacro:wheel name="rear_left"   x="0.085" y =" -0.105"/>
-    <gazebo>
+    <!-- <gazebo>
         <plugin name="diff_drive" filename="libgazebo_ros_skid_steer_drive.so">
             <updateRate>100.0</updateRate>
@@ -106,4 +108,4 @@
             <publish_wheel_tf>true</publish_wheel_tf>
         </plugin>
-    </gazebo>
+    </gazebo> -->
 </robot>

Commit message: Add files via upload

File: description/gazebo_control.xacro (robot description, xacro)
@@ -1,75 +1,22 @@
 <?xml version="1.0"?>
 <robot xmlns:xacro="http://www.ros.org/wiki/xacro">
-        <!--skid_steer_drive_controller-->
     <gazebo>
-        <plugin name="gazebo_ros_joint_state_publisher"
-            filename = "libgazebo_ros_joint_state_publisher.so">
-            <update_rate>20</update_rate>
-            <joint_name>wheel_front_left_joint</joint_name>
-            <joint_name>wheel_front_right_joint</joint_name>
-            <joint_name>wheel_rear_left_joint</joint_name>
-            <joint_name>wheel_rear_right_joint</joint_name>
-            <joint_name>wheel_rear_right_joint</joint_name>
-        </plugin>
-    </gazebo>
-    <gazebo>
-        <plugin name="gazebo_ros_joint_pose_trajectory"
-            filename = "libgazebo_ros_joint_pose_trajectory.so">
-            <update_rate>20</update_rate>
-            <joint_name>wheel_front_left_joint</joint_name>
-            <joint_name>wheel_front_right_joint</joint_name>
-            <joint_name>wheel_rear_left_joint</joint_name>
-            <joint_name>wheel_rear_right_joint</joint_name>
-            <joint_name>wheel_rear_right_joint</joint_name>
-        </plugin>
-    </gazebo>
-    <!-- <gazebo>
-        <plugin name="mobile_base_controller" filename="libgazebo_ros_skid_steer_drive.so">
-            <updateRate>100.0</updateRate>
-            <robotNamespace>/armbot</robotNamespace>
-            <leftFrontJoint>wheel_front_left_joint</leftFrontJoint>
-            <rightFrontJoint>wheel_front_right_joint</rightFrontJoint>
-            <leftRearJoint>wheel_rear_left_joint</leftRearJoint>
-            <rightRearJoint>wheel_rear_right_joint</rightRearJoint>
-            <wheelSeparation>0.16</wheelSeparation>
-            <wheelDiameter>0.085</wheelDiameter>
-            <robotBaseFrame>base_link</robotBaseFrame>
-            <torque>20</torque>
-            <commandTopic>mobile_base_controller/cmd_vel</commandTopic>
-            <odometryTopic>mobile_base_controller/odom</odometryTopic>
-            <odometryFrame>odom</odometryFrame>
+        <plugin name="skid_steer_drive" filename="libgazebo_ros_diff_drive.so">
+            <num_wheel_pairs>2</num_wheel_pairs>
+            <left_joint>wheel_front_left_joint</left_joint>
+            <right_joint>wheel_front_right_joint</right_joint>
+            <left_joint>wheel_rear_left_joint</left_joint>
+            <right_joint>wheel_rear_right_joint</right_joint>
+            <wheel_separation>0.215</wheel_separation>
+            <wheel_separation>0.215</wheel_separation>
+            <wheel_diameter>0.035</wheel_diameter>
+            <wheel_diameter>0.035</wheel_diameter>
+            <max_wheel_torque>50</max_wheel_torque>
+            <max_wheel_acceleration>10.0</max_wheel_acceleration>
+            <odometry_frame>odom</odometry_frame>
+            <robot_base_frame>base_link</robot_base_frame>
             <publish_odom>true</publish_odom>
             <publish_odom_tf>true</publish_odom_tf>
             <publish_wheel_tf>true</publish_wheel_tf>
-            <covariance_x>100.0</covariance_x>
-            <covariance_y>100.0</covariance_y>
-            <covariance_yaw>100.0</covariance_yaw>
-            <odometryRate>20.0</odometryRate>
-            <broadcastTF>true</broadcastTF>
-        </plugin>
-    </gazebo> -->
-    <gazebo>
-        <plugin name="skid_steer_drive_controller" filename="libgazebo_ros_skid_steer_drive.so">
-            <updateRate>10.0</updateRate>
-            <robotNamespace>/</robotNamespace>
-            <leftFrontJoint>left_wheel_hinge_front</leftFrontJoint>
-            <rightFrontJoint>right_wheel_hinge_front</rightFrontJoint>
-            <leftRearJoint>left_wheel_hinge_back</leftRearJoint>
-            <rightRearJoint>right_wheel_hinge_back</rightRearJoint>
-            <wheelSeparation>0.4</wheelSeparation>
-            <wheelDiameter>0.2</wheelDiameter>
-            <robotBaseFrame>robot_footprint</robotBaseFrame>
-            <torque>10</torque>
-            <topicName>cmd_vel</topicName>
-            <odometryTopic>odom</odometryTopic>
-            <odometryFrame>odom</odometryFrame>
-            <commandTopic>cmd_vel</commandTopic>
-            <topic_name_twist>cmd_vel</topic_name_twist>
-            <topic_name_odometry>odom</topic_name_odometry>
-            <topic_name_joint>joint</topic_name_joint>
-            <broadcastTF>true</broadcastTF>
-            <covariance_x>0.0001</covariance_x>
-            <covariance_y>0.0001</covariance_y>
-            <covariance_yaw>0.01</covariance_yaw>
         </plugin>
     </gazebo>

File: description/robot_core.xacro (robot description, xacro)
@@ -7,8 +7,12 @@
     <xacro:property name="base_height"   value="0.048"/>
     <xacro:property name="base_depth"    value="0.16"/>
+    <xacro:property name="wheel_constant"   value="0.08333333333333333"/>
+    <xacro:property name="wheel_mass"       value="0.5"/>
+    <xacro:property name="wheel_radius"     value="0.0425"/>
+    <xacro:property name="wheel_height"     value="0.04"/>
     <link name="chassis">
         <inertial>
             <origin xyz="0.0 0.0 0.0" rpy="0.0 0.0 0.0"/>
-            <mass value="1.0"/>
+            <mass value="5.0"/>
             <inertia
                 ixx="${base_constant * base_mass * (base_height*base_height + base_depth*base_depth)}" ixy="0.0" ixz="0.0"
@@ -81,8 +85,4 @@
         </joint>
     </xacro:macro>
-    <xacro:property name="wheel_constant"   value="0.08333333333333333"/>
-    <xacro:property name="wheel_mass"       value="0.5"/>
-    <xacro:property name="wheel_radius"     value="0.0425"/>
-    <xacro:property name="wheel_height"     value="0.04"/>
     <!-- Wheel Creating using macros -->
     <xacro:wheel name="rear_right"  x="0.085" y =" 0.105"/>
@@ -90,22 +90,3 @@
     <xacro:wheel name="front_left"  x="-0.085" y =" -0.105"/>
     <xacro:wheel name="rear_left"   x="0.085" y =" -0.105"/>
-    <!-- <gazebo>
-        <plugin name="diff_drive" filename="libgazebo_ros_skid_steer_drive.so">
-            <updateRate>100.0</updateRate>
-            <leftFrontJoint>wheel_front_left_joint</leftFrontJoint>
-            <rightFrontJoint>wheel_front_right_joint</rightFrontJoint>
-            <leftRearJoint>wheel_rear_left_joint</leftRearJoint>
-            <rightRearJoint>wheel_rear_right_joint</rightRearJoint>
-            <wheelSeparation>0.16</wheelSeparation>
-            <wheelDiameter>0.085</wheelDiameter>
-            <broadcastTF>true</broadcastTF>
-            <max_wheel_torque>200</max_wheel_torque>
-            <max_wheel_acceleration>10.0</max_wheel_acceleration>
-            <odometry_frame>odom</odometry_frame>
-            <robot_base_frame>chassis</robot_base_frame>
-            <publish_odom>true</publish_odom>
-            <publish_odom_tf>true</publish_odom_tf>
-            <publish_wheel_tf>true</publish_wheel_tf>
-        </plugin>
-    </gazebo> -->
 </robot>

Commit message: Add files via upload

File: description/gazebo_control.xacro (robot description, xacro)
@@ -1,4 +1,46 @@
 <?xml version="1.0"?>
 <robot xmlns:xacro="http://www.ros.org/wiki/xacro">
+<!--
+    <gazebo>
+        <plugin name="skid_steer_drive" filename="libgazebo_ros_diff_drive.so">
+            <num_wheel_pairs>2</num_wheel_pairs>
+            <left_joint>wheel_front_left_joint</left_joint>
+            <right_joint>wheel_front_right_joint</right_joint>
+            <left_joint>wheel_rear_left_joint</left_joint>
+            <right_joint>wheel_rear_right_joint</right_joint>
+            <wheel_separation>0.215</wheel_separation>
+            <wheel_separation>0.215</wheel_separation>
+            <wheel_diameter>0.035</wheel_diameter>
+            <wheel_diameter>0.035</wheel_diameter>
+            <max_wheel_torque>50</max_wheel_torque>
+            <max_wheel_acceleration>10.0</max_wheel_acceleration>
+            <odometry_frame>odom</odometry_frame>
+            <robot_base_frame>base_link</robot_base_frame>
+            <publish_odom>true</publish_odom>
+            <publish_odom_tf>true</publish_odom_tf>
+            <publish_wheel_tf>true</publish_wheel_tf>
+        </plugin>
+    </gazebo> -->
+<!--
+    <gazebo>
+        <plugin name="skid_steer_drive" filename="libgazebo_ros_diff_drive.so">
+            <num_wheel_pairs>2</num_wheel_pairs>
+            <left_joint>front_left_wheel_joint</left_joint>
+            <right_joint>front_right_wheel_joint</right_joint>
+            <left_joint>rear_left_wheel_joint</left_joint>
+            <right_joint>rear_right_wheel_joint</right_joint>
+            <wheel_separation>0.208</wheel_separation>
+            <wheel_separation>0.208</wheel_separation>
+            <wheel_diameter>0.080</wheel_diameter>
+            <wheel_diameter>0.080</wheel_diameter>
+            <max_wheel_torque>50</max_wheel_torque>
+            <max_wheel_acceleration>10.0</max_wheel_acceleration>
+            <odometry_frame>odom</odometry_frame>
+            <robot_base_frame>base_link</robot_base_frame>
+            <publish_odom>true</publish_odom>
+            <publish_odom_tf>true</publish_odom_tf>
+            <publish_wheel_tf>true</publish_wheel_tf>
+        </plugin>
+    </gazebo> -->
     <gazebo>
         <plugin name="skid_steer_drive" filename="libgazebo_ros_diff_drive.so">

File: description/robot_core.xacro (robot description, xacro)
@@ -77,5 +77,5 @@
         </gazebo>
         <joint name="wheel_${name}_joint" type="continuous">
-            <origin xyz="${x} ${y} -0.007" rpy="1.57 0.0 0.0"/>
+            <origin xyz="${x} ${y} -0.007" rpy="-1.57 0.0 0.0"/>
             <parent link="chassis"/>
             <child link="wheel_${name}_link"/>
@@ -85,8 +85,7 @@
         </joint>
     </xacro:macro>
-    <!-- Wheel Creating using macros -->
-    <xacro:wheel name="rear_right"  x="0.085" y =" 0.105"/>
-    <xacro:wheel name="front_right" x="-0.085" y =" 0.105"/>
-    <xacro:wheel name="front_left"  x="-0.085" y =" -0.105"/>
-    <xacro:wheel name="rear_left"   x="0.085" y =" -0.105"/>
+    <xacro:wheel name="front_left"  x="0.085" y =" 0.105"/>
+    <xacro:wheel name="rear_left" x="-0.085" y =" 0.105"/>
+    <xacro:wheel name="rear_right"  x="-0.085" y =" -0.105"/>
+    <xacro:wheel name="front_right"   x="0.085" y =" -0.105"/>
 </robot>

Commit message: Add files via upload

File: description/gazebo_control.xacro (robot description, xacro)
@@ -10,6 +10,6 @@
             <wheel_separation>0.215</wheel_separation>
             <wheel_separation>0.215</wheel_separation>
-            <wheel_diameter>0.035</wheel_diameter>
-            <wheel_diameter>0.035</wheel_diameter>
+            <wheel_diameter>0.038</wheel_diameter>
+            <wheel_diameter>0.038</wheel_diameter>
             <max_wheel_torque>50</max_wheel_torque>
             <max_wheel_acceleration>10.0</max_wheel_acceleration>

File: description/robot_core.xacro (robot description, xacro)
@@ -77,5 +77,5 @@
         </gazebo>
         <joint name="wheel_${name}_joint" type="continuous">
-            <origin xyz="${x} ${y} -0.007" rpy="-1.57 0.0 0.0"/>
+            <origin xyz="${x} ${y} -0.007" rpy="1.57 0.0 0.0"/>
             <parent link="chassis"/>
             <child link="wheel_${name}_link"/>
