Commit message: Add files via upload

File: description/gazebo_control.xacro (robot description, xacro)
@@ -2,21 +2,25 @@
 <robot xmlns:xacro="http://www.ros.org/wiki/xacro">
     <gazebo>
-        <plugin name="skid_steer_drive" filename="libgazebo_ros_diff_drive.so">
+        <plugin name="skid_steer_drive_controller" filename="libgazebo_ros_diff_drive.so">
+        <ros>
+          <argument>odom:=odom/unfiltered</argument>
+        </ros>
             <num_wheel_pairs>2</num_wheel_pairs>
-            <left_joint>wheel_front_left_joint</left_joint>
-            <right_joint>wheel_front_right_joint</right_joint>
-            <left_joint>wheel_rear_left_joint</left_joint>
-            <right_joint>wheel_rear_right_joint</right_joint>
+            <left_joint>front_left_wheel_joint</left_joint>
+            <right_joint>front_right_wheel_joint</right_joint>
+            <left_joint>rear_left_wheel_joint</left_joint>
+            <right_joint>rear_right_wheel_joint</right_joint>
             <wheel_separation>0.215</wheel_separation>
             <wheel_separation>0.215</wheel_separation>
             <wheel_diameter>0.038</wheel_diameter>
             <wheel_diameter>0.038</wheel_diameter>
-            <max_wheel_torque>50</max_wheel_torque>
+            <updateRate>100</updateRate>
+            <max_wheel_torque>1.0</max_wheel_torque>
             <max_wheel_acceleration>10.0</max_wheel_acceleration>
+            <robot_base_frame>base_footprint</robot_base_frame>
+            <publish_odom>true</publish_odom>
+            <publish_odom_tf>false</publish_odom_tf>
+            <publish_wheel_tf>true</publish_wheel_tf>
             <odometry_frame>odom</odometry_frame>
-            <robot_base_frame>base_link</robot_base_frame>
-            <publish_odom>true</publish_odom>
-            <publish_odom_tf>true</publish_odom_tf>
-            <publish_wheel_tf>true</publish_wheel_tf>
         </plugin>
     </gazebo>

File: description/lidar.xacro (robot description, xacro)
@@ -6,8 +6,8 @@
     <joint name="laser_joint" type="fixed">
         <parent link="lidar_base"/>
-        <child link="laser_frame"/>
+        <child link="laser"/>
         <origin xyz="-0.00 0.0 0.035" rpy="0.0 0.0 0.0"/>
     </joint>
-    <link name="laser_frame">
+    <link name="laser">
         <visual>
             <geometry>
@@ -27,10 +27,9 @@
         </xacro:inertial_cylinder>
     </link>
-    <gazebo reference="laser_frame">
+    <!-- <gazebo reference="laser">
         <material>Gazebo/Grey</material>
         <sensor name="laser" type="ray">
             <pose> 0 0 0 0 0 0 </pose>
             <visualize>false</visualize>
-            <!-- <visualize>true</visualize> -->
             <update_rate>10</update_rate>
             <ray>
@@ -55,4 +54,4 @@
             </plugin>
             </sensor>
-    </gazebo>
+    </gazebo> -->
 </robot>

File: description/robot.urdf.xacro (robot description, xacro)
@@ -1,13 +1,8 @@
 <?xml version="1.0"?>
 <robot xmlns:xacro="http://www.ros.org/wiki/xacro"  name="robot">
-    <xacro:arg name="use_ros2_control" default="true"/>
-    <xacro:arg name="sim_mode" default="false"/>
     <xacro:include filename="robot_core.xacro"/>
-    <xacro:if value="$(arg use_ros2_control)">
-        <xacro:include filename="ros2_control.xacro"/>
-    </xacro:if>
-    <xacro:unless value="$(arg use_ros2_control)">
-        <xacro:include filename="gazebo_control.xacro"/>
-    </xacro:unless>
+    <xacro:include filename="gazebo_control.xacro"/>
+    <!-- <xacro:include filename="ros2_control.xacro"/> -->
+    <xacro:include filename="imu.xacro"/>
     <xacro:include filename="lidar.xacro"/>
     <xacro:include filename="camera.xacro"/>

File: description/robot_core.xacro (robot description, xacro)
@@ -8,6 +8,6 @@
     <!--base_footprint -->
     <joint name="base_footprint_joint" type="fixed">
-        <parent link="base_link"/>
-        <child link="base_footprint"/>
+        <parent link="base_footprint"/>
+        <child link="base_link"/>
         <origin xyz="0 0 0" rpy="0 0 0"/>
     </joint>

File: description/ros2_control.xacro (robot description, xacro)
@@ -2,5 +2,5 @@
 <robot xmlns:xacro="http://www.ros.org/wiki/xacro">
     <xacro:macro name="define_wheel_joint" params="joint_name">
-        <joint name="wheel_${joint_name}_joint">
+        <joint name="${joint_name}_wheel_joint">
             <command_interface name="velocity">
                 <params name="min">-10.0</params>
@@ -11,39 +11,37 @@
         </joint>
     </xacro:macro>
-    <xacro:unless value="$(arg sim_mode)">
-        <ros2_control name="RealRobot" type="system">
-            <hardware>
-            <plugin>diffdrive_arduino/DiffDriveArduinoHardware</plugin>
-                <param name="wheel_front_left_joint">wheel_front_left_joint</param>
-                <param name="wheel_front_right_joint">wheel_front_right_joint</param>
-                <param name="wheel_rear_left_joint">wheel_rear_left_joint</param>
-                <param name="wheel_rear_right_joint">wheel_rear_right_joint</param>
-                <param name="loop_rate">30</param>
-                <param name="device">/dev/ttyUSB0</param>
-                <param name="baud_rate">57600</param>
-                <param name="timeout_ms">1000</param>
-                <param name="enc_counts_per_rev">19560</param>
-            </hardware>
-            <xacro:define_wheel_joint joint_name="front_left"/>
-            <xacro:define_wheel_joint joint_name="front_right"/>
-            <xacro:define_wheel_joint joint_name="rear_left"/>
-            <xacro:define_wheel_joint joint_name="rear_right"/>
-        </ros2_control>
-    </xacro:unless>
-    <xacro:if value="$(arg sim_mode)">
-        <ros2_control name="GazeboSystem" type="system">
-            <hardware>
-                <plugin>gazebo_ros2_control/GazeboSystem</plugin>
-            </hardware>
-            <xacro:define_wheel_joint joint_name="front_left"/>
-            <xacro:define_wheel_joint joint_name="front_right"/>
-            <xacro:define_wheel_joint joint_name="rear_left"/>
-            <xacro:define_wheel_joint joint_name="rear_right"/>
-        </ros2_control>
-    </xacro:if>
+    <ros2_control name="GazeboSystem" type="system">
+        <hardware>
+            <plugin>gazebo_ros2_control/GazeboSystem</plugin>
+        </hardware>
+        <xacro:define_wheel_joint joint_name="front_left"/>
+        <xacro:define_wheel_joint joint_name="front_right"/>
+        <xacro:define_wheel_joint joint_name="rear_left"/>
+        <xacro:define_wheel_joint joint_name="rear_right"/>
+    </ros2_control>
     <gazebo>
         <plugin name="gazebo_ros2_control" filename="libgazebo_ros2_control.so">
             <parameters>$(find rog_ros_bot)/config/my_controllers.yaml</parameters>
             <parameters>$(find rog_ros_bot)/config/gaz_ros2_ctl_use_sim.yaml</parameters>
+            <!-- <ros>
+                <argument>odom:=odom/unfiltered</argument>
+            </ros>
+            <num_wheel_pairs>2</num_wheel_pairs>
+            <left_joint>front_left_wheel_joint</left_joint>
+            <right_joint>front_right_wheel_joint</right_joint>
+            <left_joint>rear_left_wheel_joint</left_joint>
+            <right_joint>rear_right_wheel_joint</right_joint>
+            <wheel_separation>0.215</wheel_separation>
+            <wheel_separation>0.215</wheel_separation>
+            <wheel_diameter>0.038</wheel_diameter>
+            <wheel_diameter>0.038</wheel_diameter>
+            <updateRate>100</updateRate>
+            <max_wheel_torque>50</max_wheel_torque>
+            <max_wheel_acceleration>10.0</max_wheel_acceleration>
+            <robot_base_frame>base_footprint</robot_base_frame>
+            <publish_odom>true</publish_odom>
+            <publish_odom_tf>false</publish_odom_tf>
+            <publish_wheel_tf>true</publish_wheel_tf>
+            <odometry_frame>odom</odometry_frame> -->
         </plugin>
     </gazebo>

File: description/wheels.xacro (robot description, xacro)
@@ -3,5 +3,5 @@
     <xacro:include filename="inertial_macros.xacro"/>
     <xacro:macro name="wheel" params="name x y wheel_mass wheel_radius wheel_thickness">
-        <link name="wheel_${name}_link">
+        <link name="${name}_wheel_link">
             <visual name="">
                 <origin xyz="0.0 0.0 0.0" rpy="0.0 0.0 0.0"/>
@@ -17,5 +17,4 @@
                     <geometry>
                         <sphere radius="${wheel_radius}"/>
-                        <!-- <cylinder radius="${wheel_radius}" length="${wheel_thickness}"/> -->
                     </geometry>
             </collision>
@@ -24,10 +23,10 @@
             </xacro:inertial_cylinder>
         </link>
-        <gazebo reference = "wheel_${name}_link">
+        <gazebo reference = "${name}_wheel_link">
             <material>Gazebo/Black</material>
         </gazebo>
-        <joint name="wheel_${name}_joint" type="continuous">
+        <joint name="${name}_wheel_joint" type="continuous">
             <parent link="chassis"/>
-            <child link="wheel_${name}_link"/>
+            <child link="${name}_wheel_link"/>
             <origin xyz="${x} ${y} -0.015" rpy="-1.57 0.0 0.0"/>
             <axis xyz=".0 .0 1.0"/>
